Commit message: Made the eye pan to look straight instead of intersecting
Signed-off-by: jpmnieles <jpmnieles@connect.ust.hk>

File: urdf/grace.urdf (robot description, URDF)
Before this commit: robot robot, 10 links, 9 joints
Joints:
- joint lefteye_yaw: origin xyz=0 0.02895 0 rpy=0 0 -0.0289 -> xyz=0 0.02895 0
- joint righteye_yaw: origin xyz=0 -0.02895 0 rpy=0 0 0.0289 -> xyz=0 -0.02895 0
