Commit message: Added left and right eye cam in the chest_urdf
Signed-off-by: jpmnieles <jpmnieles@connect.ust.hk>

File: urdf/chest_grace.urdf (robot description, URDF)
Before this commit: robot robot, 9 links, 8 joints
Links:
- added link leftcamera
- added link rightcamera
Joints:
- added joint lefteye_cam: type fixed, parent lefteye, child leftcamera, origin xyz=0.015 0 0 rpy=0 0 0
- added joint righteye_cam: type fixed, parent righteye, child rightcamera, origin xyz=0.015 0 0 rpy=0 0 0
- joint torso: axis 0 -1 0 -> (none); limit lower=-1 upper=1 effort=1 velocity=1 -> (none); origin xyz=-0.12234 -0.0325 0.05692 -> xyz=-0.12234 -0.0325 0.05692 rpy=0 0 0
