Commit message: Added initial testing on the files
Signed-off-by: jpmnieles <jpmnieles@connect.ust.hk>

File: urdf/chest_grace_results.urdf (robot description, URDF)
Before this commit: robot robot, 11 links, 10 joints
Joints:
- joint eyes_pitch: origin xyz=0.0849199999999998 0.0 0.05185999999999989 rpy=3.9906374643742737e-16 0 -1.4298558473741898e-16 -> xyz=0.08492000000000018 0.0 0.05186000000000053 rpy=-1.3064604870132741e-16 0 -5.643848308639651e-17
- joint head_pitch: origin xyz=0.0 0.0 0.13171999999999967 rpy=3.9906374643742737e-16 0 -1.4298558473741898e-16 -> xyz=0.0 0.0 0.1317200000000001 rpy=-1.3064604870132741e-16 0 -5.643848308639651e-17
- joint lefteye_cam: origin xyz=0.015000000000000228 0.0 0.0 rpy=-0.2725837618652101 -0.470179129111392 -0.22861403664100136 -> xyz=0.015000000000000064 0.0 0.0 rpy=-0.4757743175985389 -0.305183729980649 -0.539632142192319
- joint lefteye_yaw: origin xyz=0.0 0.02895000000000097 0.0 rpy=3.9906374643742737e-16 0 -1.4298558473741898e-16 -> xyz=0.0 0.028950000000000253 0.0 rpy=-1.3064604870132741e-16 0 -5.643848308639651e-17
- joint neck_pitch: origin xyz=0.0 0.0 0.0 rpy=3.9906374643742737e-16 0 -1.4298558473741898e-16 -> xyz=0.0 0.0 0.0 rpy=-1.3064604870132741e-16 0 -5.643848308639651e-17
- joint neck_yaw: origin xyz=0.0 0.0 0.0 rpy=3.9906374643742737e-16 0 -1.4298558473741898e-16 -> xyz=0.0 0.0 0.0 rpy=-1.3064604870132741e-16 0 -5.643848308639651e-17
- joint righteye_cam: origin xyz=0.014999999999999803 0.0 0.0 rpy=0.3793764370910186 -0.4250905711033968 0.05414172136937682 -> xyz=0.015000000000000251 0.0 0.0 rpy=0.44803016476492735 -0.2849255765358385 0.27326619540272046
- joint righteye_yaw: origin xyz=0.0 -0.02895000000000043 0.0 rpy=3.9906374643742737e-16 0 -1.4298558473741898e-16 -> xyz=0.0 -0.028950000000000028 0.0 rpy=-1.3064604870132741e-16 0 -5.643848308639651e-17
- joint torso: origin xyz=-0.12233999999999948 -0.03250000000000028 0.05691999999999999 rpy=0.0 0.0 0.0 -> xyz=-0.12234000000000009 -0.032499999999999925 0.056919999999999804 rpy=0.0 0.0 0.0
