Commit message: Corrected the positioning of the realsense camera
Signed-off-by: jpmnieles <jpmnieles@connect.ust.hk>

File: urdf/chest_grace_cam.urdf (robot description, URDF)
Before this commit: robot robot, 11 links, 10 joints
Links:
- link realsense: geometry visual box size=0.09 0.025 0.025
Joints:
- joint torso: origin xyz=-0.0325 -0.05692 -0.12234 rpy=1.5708 -1.5708 0 -> xyz=0.0325 -0.05692 -0.12234 rpy=1.5708 -1.5708 0
