Commit message: Updated the values of the marked urdf
Signed-off-by: jpmnieles <jpmnieles@connect.ust.hk>

File: urdf/chest_grace_marked.urdf (robot description, URDF)
Before this commit: robot robot, 11 links, 10 joints
Links:
- link realsense: geometry visual box size=0.09 0.025 0.025
Joints:
- joint chest_camera: origin xyz=0 0 0.44739 rpy=0 0 0 -> xyz=0 0 0.44739 rpy=-1.5708 0 -1.5708
- joint lefteye_cam: origin xyz=*0.015 0 0 rpy=*0 *0 *0 -> xyz=*0.015 0 0 rpy=*-1.5708 *0 *-1.5708
- joint righteye_cam: origin xyz=*0.015 0 0 rpy=*0 *0 *0 -> xyz=*0.015 0 0 rpy=*-1.5708 *0 *-1.5708
- joint torso: origin xyz=*-0.12234 *-0.0325 *0.05692 rpy=0 0 0 -> xyz=*0.0325 *-0.05692 *-0.12234 rpy=1.5708 -1.5708 0
