Commit message: Changed the neck pitch axis and explicitly added rpy origin
Signed-off-by: jpmnieles <jpmnieles@connect.ust.hk>

File: urdf/chest_grace_cam_true.urdf (robot description, URDF)
Before this commit: robot robot, 11 links, 10 joints
Joints:
- joint eyes_pitch: origin xyz=0.08492 0 0.05186 -> xyz=0.08492 0 0.05186 rpy=0 0 0
- joint head_pitch: origin xyz=0 0 0.13172 -> xyz=0 0 0.13172 rpy=0 0 0
- joint lefteye_yaw: origin xyz=0 0.02895 0 -> xyz=0 0.02895 0 rpy=0 0 0
- joint neck_pitch: axis 0 -1 0 -> 0 1 0; origin xyz=0 0 0 -> xyz=0 0 0 rpy=0 0 0
- joint neck_yaw: origin xyz=0 0 0 -> xyz=0 0 0 rpy=0 0 0
- joint righteye_yaw: origin xyz=0 -0.02895 0 -> xyz=0 -0.02895 0 rpy=0 0 0

Commit message: Changed the radius of the eye for visualization
Signed-off-by: jpmnieles <jpmnieles@connect.ust.hk>

File: urdf/chest_grace_cam_true.urdf (robot description, URDF)
Before this commit: robot robot, 11 links, 10 joints
Links:
- link lefteye: geometry visual sphere radius=0.015
- link righteye: geometry visual sphere radius=0.015
